Commit message: Add Phase 2B: YOLO + depth centroid vision-based pick-and-place (v1.1)
Detector:
- yolo_detector.py: YOLOv8 inference with HSV colour fallback for Gazebo geometry
- Depth back-projection: (u,v,depth) → camera optical frame → world frame
- Same /detected_pose topic interface as Phase 2A — orchestrator unchanged
- pick_place_demo.launch.py: detector:=yolo / detector:=apriltag launch arg

Infrastructure fixes:
- panda.urdf.xacro: add world link + world_joint to anchor robot in Gazebo physics
- gazebo.launch.py: spawn hand_trajectory_controller (JointTrajectoryController)
- ros2_controllers.yaml: remove panda_finger_joint2 from controller joints
  (mimic joint — gz_ros2_control handles it internally, no command interface)
- pick_place.sdf: add red_box_plain (uniformly red, no AprilTag texture) for YOLO

pick_place_node.py improvements:
- Gripper via direct JointTrajectory topic publish — bypasses MoveIt2 start-state
  bounds check (joint2 driven negative by gz_ros2_control mimic) and avoids
  rclpy ActionClient executor thread conflicts
- Grasp height: fingertips target box midpoint (tag.z - BOX_HALF_HEIGHT + HAND_LENGTH)
- Release sequence: detach → open → 1s physics settle → retreat

Co-Authored-By: Claude Sonnet 4.6 <noreply@anthropic.com>

File: ros2_ws/src/arm_bringup/urdf/panda.urdf.xacro (robot description, xacro)
@@ -3,4 +3,11 @@
     <xacro:arg name="initial_positions_file" default="$(find arm_bringup)/config/initial_positions.yaml" />
     <xacro:arg name="ros2_control_hardware_type" default="mock_components" />
+    <!-- Fix robot base to world so Gazebo doesn't apply gravity to the base link -->
+    <link name="world"/>
+    <joint name="world_joint" type="fixed">
+        <parent link="world"/>
+        <child link="panda_link0"/>
+        <origin xyz="0 0 0" rpy="0 0 0"/>
+    </joint>
     <!-- Import panda urdf file -->
     <xacro:include filename="$(find moveit_resources_panda_description)/urdf/panda.urdf.xacro" />
